File: pandp.sch (KiCad schematic (older format))
At the start: 89 parts, among them IC1 ADP2303-5, P1 CONN_01X02, P10 CONN_01X04, P11 CONN_01X02, P12 CONN_02X04, P13 CONN_01X02, P14 CONN_01X04, P15 CONN_01X04, P16 CONN_01X03, P17 CONN_01X03, P18 CONN_01X03, P19 CONN_01X03, P2 CONN_01X03, P20 CONN_01X03, P21 CONN_01X03, P22 CONN_02X03, P23 CONN_02X03, P24 CONN_02X03, P25 CONN_02X03, P26 CONN_01X03, P27 CONN_01X03, P28 CONN_01X03, P29 CONN_01X03, P3 CONN_01X02, P30 CONN_01X04, P31 CONN_01X04, P32 CONN_01X04, P33 CONN_01X04, P4 CONN_01X03, P6 CONN_01X03, P7 CONN_01X03, P8 USB_OTG, P9 CONN_01X02, Q1 IRF540N, Q2 IRF540N, SW1 SW_PUSH, U1 AP1117D33, U2 STM32F103RC, Y1 Crystal_Small - 2101357 on el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, Y2 Crystal_Small - 2063972 on el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

Commit message: first autorouter - dont like
Parts:
- removed C11, C7: CP, SMD_Packages:SMD-1210_Pol, symbol CP
- added R24: R, Resistors_SMD:R_0402, symbol R
Connections:
- net +5V: now also R24.2; no longer P8.1 (VCC)
- net GND: no longer C12.2, C13.2, C4.2, C6.2
- net GNDD: now also C12.2, C13.2, C4.2, C6.2
- new net +5VL: P8.1 (VCC), R24.1
Other:
- moved on the sheet: C5, C9
Changed lines of the file:
@@
 LIBS:MyConnectors
 LIBS:pandp-cache
-LIBS:mls-cache
 EELAYER 25 0
 EELAYER END
@@
 L C C5
 U 1 1 57F1F5A1
-P 1650 5100
-F 0 "C5" H 1675 5200 50  0000 L CNN
-F 1 "C" H 1675 5000 50  0000 L CNN
-F 2 "Capacitors_SMD:C_0805_HandSoldering" H 1688 4950 50  0001 C CNN
-F 3 "" H 1650 5100 50  0000 C CNN
-	1    1650 5100
+P 1800 5100
+F 0 "C5" H 1825 5200 50  0000 L CNN
+F 1 "C" H 1825 5000 50  0000 L CNN
+F 2 "Capacitors_SMD:C_0805_HandSoldering" H 1838 4950 50  0001 C CNN
+F 3 "" H 1800 5100 50  0000 C CNN
+	1    1800 5100
 	1    0    0    -1
 $EndComp
@@
 L C C9
 U 1 1 57F1F5A2
-P 2350 5100
-F 0 "C9" H 2375 5200 50  0000 L CNN
-F 1 "C" H 2375 5000 50  0000 L CNN
-F 2 "Capacitors_SMD:C_0805_HandSoldering" H 2388 4950 50  0001 C CNN
-F 3 "" H 2350 5100 50  0000 C CNN
-	1    2350 5100
+P 2500 5100
+F 0 "C9" H 2525 5200 50  0000 L CNN
+F 1 "C" H 2525 5000 50  0000 L CNN
+F 2 "Capacitors_SMD:C_0805_HandSoldering" H 2538 4950 50  0001 C CNN
+F 3 "" H 2500 5100 50  0000 C CNN
+	1    2500 5100
 	1    0    0    -1
 $EndComp
@@
 F 3 "" H 850 5100 50  0000 C CNN
 	1    850  5100
-	1    0    0    -1
-$EndComp
-$Comp
-L CP C7
-U 1 1 57F1F5A4
-P 1950 5100
-F 0 "C7" H 1975 5200 50  0000 L CNN
-F 1 "CP" H 1975 5000 50  0000 L CNN
-F 2 "SMD_Packages:SMD-1210_Pol" H 1988 4950 50  0001 C CNN
-F 3 "" H 1950 5100 50  0000 C CNN
-	1    1950 5100
-	1    0    0    -1
-$EndComp
-$Comp
-L CP C11
-U 1 1 57F1F5A5
-P 2650 5100
-F 0 "C11" H 2675 5200 50  0000 L CNN
-F 1 "CP" H 2675 5000 50  0000 L CNN
-F 2 "SMD_Packages:SMD-1210_Pol" H 2688 4950 50  0001 C CNN
-F 3 "" H 2650 5100 50  0000 C CNN
-	1    2650 5100
 	1    0    0    -1
 $EndComp
@@
 	0    1    1    0
 $EndComp
-$Comp
-L GND #PWR038
-U 1 1 57F3320D
-P 3250 9600
-F 0 "#PWR038" H 3250 9350 50  0001 C CNN
-F 1 "GND" H 3250 9450 50  0000 C CNN
-F 2 "" H 3250 9600 50  0000 C CNN
-F 3 "" H 3250 9600 50  0000 C CNN
-	1    3250 9600
-	-1   0    0    1
-$EndComp
 Text GLabel 1250 10500 3    60   Input ~ 0
 OSC32_OUT
@@
 	1    1750 9800
 	0    1    1    0
-$EndComp
-$Comp
-L GND #PWR039
-U 1 1 57F33210
-P 1500 9600
-F 0 "#PWR039" H 1500 9350 50  0001 C CNN
-F 1 "GND" H 1500 9450 50  0000 C CNN
-F 2 "" H 1500 9600 50  0000 C CNN
-F 3 "" H 1500 9600 50  0000 C CNN
-	1    1500 9600
-	-1   0    0    1
-$EndComp
-$Comp
-L +5V #PWR040
-U 1 1 57F33217
-P 4200 1750
-F 0 "#PWR040" H 4200 1600 50  0001 C CNN
-F 1 "+5V" H 4200 1890 50  0000 C CNN
-F 2 "" H 4200 1750 50  0000 C CNN
-F 3 "" H 4200 1750 50  0000 C CNN
-	1    4200 1750
-	-1   0    0    1
 $EndComp
 Text GLabel 6450 4950 0    60   Input ~ 0
@@
 BOOT0
 $Comp
-L +3.3V #PWR041
+L +3.3V #PWR038
 U 1 1 57F33218
 P 10700 8500
-F 0 "#PWR041" H 10700 8350 50  0001 C CNN
+F 0 "#PWR038" H 10700 8350 50  0001 C CNN
 F 1 "+3.3V" H 10700 8640 50  0000 C CNN
 F 2 "" H 10700 8500 50  0000 C CNN
@@
 $EndComp
 $Comp
-L GND #PWR042
+L GND #PWR039
 U 1 1 57F3740F
 P 1000 6450
-F 0 "#PWR042" H 1000 6200 50  0001 C CNN
+F 0 "#PWR039" H 1000 6200 50  0001 C CNN
 F 1 "GND" H 1000 6300 50  0000 C CNN
 F 2 "" H 1000 6450 50  0000 C CNN
@@
 $EndComp
 $Comp
-L GND #PWR043
+L GND #PWR040
 U 1 1 57F3A4BF
 P 2450 6850
-F 0 "#PWR043" H 2450 6600 50  0001 C CNN
+F 0 "#PWR040" H 2450 6600 50  0001 C CNN
 F 1 "GND" H 2450 6700 50  0000 C CNN
 F 2 "" H 2450 6850 50  0000 C CNN
@@
 Connection ~ 1000 5250
 Wire Wire Line
-	1650 5250 1950 5250
-Wire Wire Line
-	1650 4950 1950 4950
-Wire Wire Line
 	1800 4850 1800 4950
-Connection ~ 1800 4950
 Wire Wire Line
 	1800 5250 1800 5350
-Connection ~ 1800 5250
-Wire Wire Line
-	2350 5250 2650 5250
-Wire Wire Line
-	2350 4950 2650 4950
 Wire Wire Line
 	2500 4850 2500 4950
-Connection ~ 2500 4950
 Wire Wire Line
 	2500 5250 2500 5350
-Connection ~ 2500 5250
 Wire Wire Line
 	1000 2650 1000 2800
@@
 	6450 3550 6800 3550
 $Comp
-L +3.3V #PWR045
+L +3.3V #PWR041
 U 1 1 57F410C2
 P 7450 2850
-F 0 "#PWR045" H 7450 2700 50  0001 C CNN
+F 0 "#PWR041" H 7450 2700 50  0001 C CNN
 F 1 "+3.3V" H 7450 2990 50  0000 C CNN
 F 2 "" H 7450 2850 50  0000 C CNN
@@
 $EndComp
 $Comp
-L GND #PWR046
+L GND #PWR042
 U 1 1 57F42396
 P 4100 10550
-F 0 "#PWR046" H 4100 10300 50  0001 C CNN
+F 0 "#PWR042" H 4100 10300 50  0001 C CNN
 F 1 "GND" H 4100 10400 50  0000 C CNN
 F 2 "" H 4100 10550 50  0000 C CNN
@@
 RESET
 $Comp
-L +3.3V #PWR047
+L +3.3V #PWR043
 U 1 1 57F427F5
 P 5600 10550
-F 0 "#PWR047" H 5600 10400 50  0001 C CNN
+F 0 "#PWR043" H 5600 10400 50  0001 C CNN
 F 1 "+3.3V" H 5600 10690 50  0000 C CNN
 F 2 "" H 5600 10550 50  0000 C CNN
@@
 $EndComp
 $Comp
-L GND #PWR048
+L GND #PWR044
 U 1 1 57F4CF5F
 P 7000 2150
-F 0 "#PWR048" H 7000 1900 50  0001 C CNN
+F 0 "#PWR044" H 7000 1900 50  0001 C CNN
 F 1 "GND" H 7000 2000 50  0000 C CNN
 F 2 "" H 7000 2150 50  0000 C CNN
@@
 Connection ~ 7200 1650
 $Comp
-L +3.3V #PWR049
+L +3.3V #PWR045
 U 1 1 57F4E376
 P 7200 1250
-F 0 "#PWR049" H 7200 1100 50  0001 C CNN
+F 0 "#PWR045" H 7200 1100 50  0001 C CNN
 F 1 "+3.3V" H 7200 1390 50  0000 C CNN
 F 2 "" H 7200 1250 50  0000 C CNN
@@
 $EndComp
 $Comp
-L GND #PWR050
+L GND #PWR046
 U 1 1 57F4ED8F
 P 7800 2150
-F 0 "#PWR050" H 7800 1900 50  0001 C CNN
+F 0 "#PWR046" H 7800 1900 50  0001 C CNN
 F 1 "GND" H 7800 2000 50  0000 C CNN
 F 2 "" H 7800 2150 50  0000 C CNN
@@
 Connection ~ 8000 1650
 $Comp
-L +3.3V #PWR051
+L +3.3V #PWR047
 U 1 1 57F4EDA3
 P 8000 1250
-F 0 "#PWR051" H 8000 1100 50  0001 C CNN
+F 0 "#PWR047" H 8000 1100 50  0001 C CNN
 F 1 "+3.3V" H 8000 1390 50  0000 C CNN
 F 2 "" H 8000 1250 50  0000 C CNN
@@
 USB_D-
 $Comp
-L +12V #PWR052
+L +12V #PWR048
 U 1 1 57F6094B
 P 850 1700
-F 0 "#PWR052" H 850 1550 50  0001 C CNN
+F 0 "#PWR048" H 850 1550 50  0001 C CNN
 F 1 "+12V" H 850 1840 50  0000 C CNN
 F 2 "" H 850 1700 50  0000 C CNN
@@
 $EndComp
 $Comp
-L +12V #PWR053
+L +12V #PWR049
 U 1 1 57F6141B
 P 1000 2650
-F 0 "#PWR053" H 1000 2500 50  0001 C CNN
+F 0 "#PWR049" H 1000 2500 50  0001 C CNN
 F 1 "+12V" H 1000 2790 50  0000 C CNN
 F 2 "" H 1000 2650 50  0000 C CNN
@@
 $EndComp
 $Comp
-L +12V #PWR054
+L +12V #PWR050
 U 1 1 57F615DA
 P 1000 4850
-F 0 "#PWR054" H 1000 4700 50  0001 C CNN
+F 0 "#PWR050" H 1000 4700 50  0001 C CNN
 F 1 "+12V" H 1000 4990 50  0000 C CNN
 F 2 "" H 1000 4850 50  0000 C CNN
@@
 $EndComp
 $Comp
-L GNDD #PWR055
+L GNDD #PWR051
 U 1 1 57F61C8F
 P 7800 7250
-F 0 "#PWR055" H 7800 7000 50  0001 C CNN
+F 0 "#PWR051" H 7800 7000 50  0001 C CNN
 F 1 "GNDD" H 7800 7100 50  0000 C CNN
 F 2 "" H 7800 7250 50  0000 C CNN
@@
 $EndComp
 $Comp
-L GNDD #PWR056
+L GNDD #PWR052
 U 1 1 57F634A7
 P 4400 2750
-F 0 "#PWR056" H 4400 2500 50  0001 C CNN
+F 0 "#PWR052" H 4400 2500 50  0001 C CNN
 F 1 "GNDD" H 4400 2600 50  0000 C CNN
 F 2 "" H 4400 2750 50  0000 C CNN
@@
 $EndComp
 $Comp
-L GND #PWR057
+L GND #PWR053
 U 1 1 57F63E20
 P 4100 2750
-F 0 "#PWR057" H 4100 2500 50  0001 C CNN
+F 0 "#PWR053" H 4100 2500 50  0001 C CNN
 F 1 "GND" H 4100 2600 50  0000 C CNN
 F 2 "" H 4100 2750 50  0000 C CNN
@@
 $EndComp
 $Comp
-L GND #PWR058
+L GND #PWR054
 U 1 1 57F65296
 P 1600 3650
-F 0 "#PWR058" H 1600 3400 50  0001 C CNN
+F 0 "#PWR054" H 1600 3400 50  0001 C CNN
 F 1 "GND" H 1600 3500 50  0000 C CNN
 F 2 "" H 1600 3650 50  0000 C CNN
@@
 $EndComp
 $Comp
-L GND #PWR059
+L GND #PWR055
 U 1 1 57F65B7A
 P 4100 3000
-F 0 "#PWR059" H 4100 2750 50  0001 C CNN
+F 0 "#PWR055" H 4100 2750 50  0001 C CNN
 F 1 "GND" H 4100 2850 50  0000 C CNN
 F 2 "" H 4100 3000 50  0000 C CNN
@@
 $EndComp
 $Comp
-L GNDA #PWR060
+L GNDA #PWR056
 U 1 1 57F66063
 P 4400 3000
-F 0 "#PWR060" H 4400 2750 50  0001 C CNN
+F 0 "#PWR056" H 4400 2750 50  0001 C CNN
 F 1 "GNDA" H 4400 2850 50  0000 C CNN
 F 2 "" H 4400 3000 50  0000 C CNN
@@
 $EndComp
 $Comp
-L GNDA #PWR061
+L GNDA #PWR057
 U 1 1 57F661DA
 P 4300 850
-F 0 "#PWR061" H 4300 600 50  0001 C CNN
+F 0 "#PWR057" H 4300 600 50  0001 C CNN
 F 1 "GNDA" H 4300 700 50  0000 C CNN
 F 2 "" H 4300 850 50  0000 C CNN
@@
 $EndComp
 $Comp
-L +5V #PWR062
+L +5V #PWR058
 U 1 1 57F66656
 P 850 850
-F 0 "#PWR062" H 850 700 50  0001 C CNN
+F 0 "#PWR058" H 850 700 50  0001 C CNN
 F 1 "+5V" H 850 990 50  0000 C CNN
 F 2 "" H 850 850 50  0000 C CNN
@@
 5V_IND
 $Comp
-L +12V #PWR?
+L +12V #PWR059
 U 1 1 57F67DAB
 P 2300 6950
-F 0 "#PWR?" H 2300 6800 50  0001 C CNN
+F 0 "#PWR059" H 2300 6800 50  0001 C CNN
 F 1 "+12V" H 2300 7090 50  0000 C CNN
 F 2 "" H 2300 6950 50  0000 C CNN
@@
 	1    0    0    -1
 $EndComp
+$Comp
+L GNDD #PWR060
+U 1 1 57F5E959
+P 1500 9600
+F 0 "#PWR060" H 1500 9350 50  0001 C CNN
+F 1 "GNDD" H 1500 9450 50  0000 C CNN
+F 2 "" H 1500 9600 50  0000 C CNN
+F 3 "" H 1500 9600 50  0000 C CNN
+	1    1500 9600
+	-1   0    0    1
+$EndComp
+$Comp
+L GNDD #PWR061
+U 1 1 57F5EA6F
+P 3250 9600
+F 0 "#PWR061" H 3250 9350 50  0001 C CNN
+F 1 "GNDD" H 3250 9450 50  0000 C CNN
+F 2 "" H 3250 9600 50  0000 C CNN
+F 3 "" H 3250 9600 50  0000 C CNN
+	1    3250 9600
+	-1   0    0    1
+$EndComp
+$Comp
+L R R24
+U 1 1 57F674AD
+P 4250 3300
+F 0 "R24" V 4330 3300 50  0000 C CNN
+F 1 "R" V 4250 3300 50  0000 C CNN
+F 2 "Resistors_SMD:R_0402" V 4180 3300 50  0001 C CNN
+F 3 "" H 4250 3300 50  0000 C CNN
+	1    4250 3300
+	0    -1   -1   0
+$EndComp
+$Comp
+L +5V #PWR062
+U 1 1 57F675CA
+P 4400 3300
+F 0 "#PWR062" H 4400 3150 50  0001 C CNN
+F 1 "+5V" H 4400 3440 50  0000 C CNN
+F 2 "" H 4400 3300 50  0000 C CNN
+F 3 "" H 4400 3300 50  0000 C CNN
+	1    4400 3300
+	0    1    1    0
+$EndComp
+$Comp
+L +5VL #PWR063
+U 1 1 57F676E2
+P 4100 3300
+F 0 "#PWR063" H 4100 3150 50  0001 C CNN
+F 1 "+5VL" H 4100 3440 50  0000 C CNN
+F 2 "" H 4100 3300 50  0000 C CNN
+F 3 "" H 4100 3300 50  0000 C CNN
+	1    4100 3300
+	0    -1   -1   0
+$EndComp
+$Comp
+L +5VL #PWR064
+U 1 1 57F67855
+P 4200 1750
+F 0 "#PWR064" H 4200 1600 50  0001 C CNN
+F 1 "+5VL" H 4200 1890 50  0000 C CNN
+F 2 "" H 4200 1750 50  0000 C CNN
+F 3 "" H 4200 1750 50  0000 C CNN
+	1    4200 1750
+	-1   0    0    1
+$EndComp
 $EndSCHEMATC
